Commit message: yumi_pc versions

File: yumi_description/urdf/yumi.urdf.xacro (robot description, xacro)
@@ -9,4 +9,6 @@
 	<!--Import the yumi servo gripper macro -->
 	<xacro:include filename="$(find yumi_description)/urdf/Grippers/yumi_servo_gripper.xacro"/>
+	<!--Import the yumi optodaq sensors macro -->
+	<xacro:include filename="$(find yumi_description)/urdf/Extras/yumi_optodaq_sensors.xacro"/>
 	<!-- Import Gazebo plugins -->
 	<xacro:include filename="$(find yumi_description)/urdf/Gazebo/gazebo.urdf.xacro"/>
@@ -15,12 +17,18 @@
 		<origin xyz="0 0 0.1" rpy="0 0 0" />
 	</xacro:yumi>
-	<!--right gripper-->
-	<xacro:yumi_servo_gripper name="gripper_r" hardware_interface="hardware_interface/$(arg grippers_interface)" parent="yumi_link_7_r">
-		<origin xyz="0 0 0.007" rpy="0 0 ${PI}" />
-	</xacro:yumi_servo_gripper>
-	<!--left gripper-->
-	<xacro:yumi_servo_gripper name="gripper_l" hardware_interface="hardware_interface/$(arg grippers_interface)" parent="yumi_link_7_l">
-		<origin xyz="0 0 0.007" rpy="0 0 ${PI}" />
-	</xacro:yumi_servo_gripper>
+  <xacro:yumi_optodaq_sensor name="optodaq_r" parent="yumi_link_7_r">
+      <origin xyz="0 0 0.033" rpy="0 0 ${-PI/4}" />
+  </xacro:yumi_optodaq_sensor>
+  <xacro:yumi_optodaq_sensor name="optodaq_l" parent="yumi_link_7_l">
+	  <origin xyz="0 0 0.033" rpy="0 0 ${-PI/4}" />
+  </xacro:yumi_optodaq_sensor>
+  <!--right gripper-->
+  <xacro:yumi_servo_gripper name="gripper_r" hardware_interface="hardware_interface/EffortJointInterface" parent="optodaq_r_sensor_link">
+    <origin xyz="0 0 0.033" rpy="0 0.0 ${PI/4}" />
+  </xacro:yumi_servo_gripper>
+  <!--left gripper-->
+  <xacro:yumi_servo_gripper name="gripper_l" hardware_interface="hardware_interface/EffortJointInterface" parent="optodaq_l_sensor_link">
+    <origin xyz="0 0 0.033" rpy="0 0.0 ${PI/4}" />
+  </xacro:yumi_servo_gripper>
         <!--
 	<xacro:property name="yumi_setup" value="$(arg yumi_setup)" />
